File: Schematics/RadHardSchematics 2/RadHardSchematics.kicad_sch (KiCad schematic)
At the start: 33 parts, among them U1 74CBTLV3257, U10 CAT24C 512XHM, U11 AT24CS01-SSHM, U12 AT24CS32-SSHM, U13 CAT24C128 SSHM, U14 AT24CS01-SSHM, U15 AT24CS32-SSHM, U16 CAT24C128 SSHM, U17 AT24CS01-XHM, U18 AT24CS32-XHM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

Commit message: latest pcb push
Parts:
- R10, R11, R12, R13, R14, R15, R4, R5, R6, R9: footprint Resistor_SMD:R_4020_10251Metric_Pad1.65x5.30mm_HandSolder -> Resistor_SMD:R_0805_2012Metric
Changed lines of the file:
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@@
       (effects (font (size 1.27 1.27)) (justify right))
     )
-    (property "Footprint" "Resistor_SMD:R_4020_10251Metric_Pad1.65x5.30mm_HandSolder" (at 101.854 100.076 90)
+    (property "Footprint" "Resistor_SMD:R_0805_2012Metric" (at 101.854 100.076 90)
       (effects (font (size 1.27 1.27)) hide)
     )
@@
       (effects (font (size 1.27 1.27)))
     )
-    (property "Footprint" "Resistor_SMD:R_4020_10251Metric_Pad1.65x5.30mm_HandSolder" (at 127.254 30.734 90)
+    (property "Footprint" "Resistor_SMD:R_0805_2012Metric" (at 127.254 30.734 90)
       (effects (font (size 1.27 1.27)) hide)
     )
@@
       (effects (font (size 1.27 1.27)) (justify right))
     )
-    (property "Footprint" "Resistor_SMD:R_4020_10251Metric_Pad1.65x5.30mm_HandSolder" (at 81.534 100.076 90)
+    (property "Footprint" "Resistor_SMD:R_0805_2012Metric" (at 81.534 100.076 90)
       (effects (font (size 1.27 1.27)) hide)
     )
@@
       (effects (font (size 1.27 1.27)))
     )
-    (property "Footprint" "Resistor_SMD:R_4020_10251Metric_Pad1.65x5.30mm_HandSolder" (at 127.254 21.844 90)
+    (property "Footprint" "Resistor_SMD:R_0805_2012Metric" (at 127.254 21.844 90)
       (effects (font (size 1.27 1.27)) hide)
     )
@@
       (effects (font (size 1.27 1.27)))
     )
-    (property "Footprint" "Resistor_SMD:R_4020_10251Metric_Pad1.65x5.30mm_HandSolder" (at 127.254 37.084 90)
+    (property "Footprint" "Resistor_SMD:R_0805_2012Metric" (at 127.254 37.084 90)
       (effects (font (size 1.27 1.27)) hide)
     )
@@
       (effects (font (size 1.27 1.27)) (justify right))
     )
-    (property "Footprint" "Resistor_SMD:R_4020_10251Metric_Pad1.65x5.30mm_HandSolder" (at 67.564 100.076 90)
+    (property "Footprint" "Resistor_SMD:R_0805_2012Metric" (at 67.564 100.076 90)
       (effects (font (size 1.27 1.27)) hide)
     )
@@
       (effects (font (size 1.27 1.27)))
     )
-    (property "Footprint" "Resistor_SMD:R_4020_10251Metric_Pad1.65x5.30mm_HandSolder" (at 127.254 26.924 90)
+    (property "Footprint" "Resistor_SMD:R_0805_2012Metric" (at 127.254 26.924 90)
       (effects (font (size 1.27 1.27)) hide)
     )
@@
       (effects (font (size 1.27 1.27)))
     )
-    (property "Footprint" "Resistor_SMD:R_4020_10251Metric_Pad1.65x5.30mm_HandSolder" (at 127.254 40.894 90)
+    (property "Footprint" "Resistor_SMD:R_0805_2012Metric" (at 127.254 40.894 90)
       (effects (font (size 1.27 1.27)) hide)
     )
@@
       (effects (font (size 1.27 1.27)))
     )
-    (property "Footprint" "Resistor_SMD:R_4020_10251Metric_Pad1.65x5.30mm_HandSolder" (at 127.254 19.304 90)
+    (property "Footprint" "Resistor_SMD:R_0805_2012Metric" (at 127.254 19.304 90)
       (effects (font (size 1.27 1.27)) hide)
     )
@@
       (effects (font (size 1.27 1.27)) (justify right))
     )
-    (property "Footprint" "Resistor_SMD:R_4020_10251Metric_Pad1.65x5.30mm_HandSolder" (at 75.184 100.076 90)
-      (effects (font (size 1.27 1.27)) hide)
-    )
+    (property "Footprint" "Resistor_SMD:R_0805_2012Metric" (at 75.184 100.076 90)
+      (effects (font (size 1.27 1.27)) hide)
+    )
