File: RadHardSchematicsNewest/RadHardSchematics.kicad_pcb (KiCad board)
At the start: 2 copper layers, 142.5 x 79.8 mm, 33 parts, among them U1 74CBTLV3257, U10 CAT24C 512XHM, U11 AT24CS01-SSHM, U12 AT24CS32-SSHM, U13 CAT24C128 SSHM, U14 AT24CS01-SSHM, U15 AT24CS32-SSHM, U16 CAT24C128 SSHM, U17 AT24CS01-XHM, U18 AT24CS32-XHM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

Commit message: Changed Footprints for New PCB
Parts:
- U1, U2: footprint Package_SO:SO-16_3.9x9.9mm_P1.27mm -> Package_SO:TSSOP-16_4.4x5mm_P0.65mm
- U13, U16, U7, U8: footprint Package_SO:SOIC-8-1EP_3.9x4.9mm_P1.27mm_EP2.29x3mm -> Package_SO:SOIC-8_3.9x4.9mm_P1.27mm
- moved U1 3.12 mm to (78.4, 52.6)
- moved R5 1.76 mm to (78.8, 45.4)
- moved U2 0.98 mm to (78.5, 67.4)
Routing:
- net +3V3: track 42.5 -> 17.5 mm
- net Net-(A2-SCL/A5-Pad32): track 25.0 -> 33.2 mm, vias 2 -> 4
- net Net-(A2-SDA/A4-Pad31): track 23.9 -> 28.7 mm
- net Net-(R9-Pad2): track 19.0 -> 23.4 mm
- net Net-(U10-SCL): track 228.6 -> 225.4 mm
- net Net-(R6-Pad2): track 38.4 -> 41.0 mm
- net Net-(U10-SDA): track 373.5 -> 376.1 mm
- net Net-(A2-D13): track 20.0 -> 22.3 mm
- net Net-(A2-D12): track 10.1 -> 11.5 mm
- net Net-(U12-SCL): track 240.0 -> 239.0 mm
- net Net-(U3-SDA): vias 2 -> 0
